File: MCU.sch (KiCad schematic (older format))
At the start: 67 parts, among them J12 USB_B_Mini, J13 Micro_SD_Card, J55 Conn_02x20_Odd_Even, SW1 SW_Push, U1 STM32F407IGTx, U7 24C02, Y1 12MHz, 20pF

Commit message: associated more footprints
Parts:
- C1, C3, C33, C34: footprint (none) -> Capacitor_SMD:C_0603_1608Metric_Pad1.05x0.95mm_HandSolder
- C19, C4: footprint (none) -> Capacitor_SMD:C_0805_2012Metric_Pad1.15x1.40mm_HandSolder
- EXP1, EXP2: footprint (none) -> Connector_PinHeader_2.54mm:PinHeader_2x05_P2.54mm_Vertical
- F5: footprint (none) -> Fuse:Fuse_1206_3216Metric_Pad1.42x1.75mm_HandSolder
- I2C1, UART1: footprint (none) -> Connector_PinHeader_2.54mm:PinHeader_1x04_P2.54mm_Vertical
- J12: footprint (none) -> Connector_USB:USB_Mini-B_Wuerth_65100516121_Horizontal
- J13: footprint (none) -> Connector_Card:microSD_HC_Wuerth_693072010801
- J55: footprint (none) -> Connector_PinHeader_2.54mm:PinHeader_2x20_P2.54mm_Vertical
- JP1, JP2: footprint (none) -> Connector_PinHeader_2.54mm:PinHeader_1x02_P2.54mm_Vertical
- SPI1: footprint (none) -> Connector_PinHeader_2.54mm:PinHeader_2x03_P2.54mm_Vertical
- SWD1: footprint (none) -> Connector_PinHeader_2.54mm:PinHeader_1x05_P2.54mm_Vertical
Changed lines of the file:
@@
 F 0 "C4" V 8958 762 39  0000 R TNN
 F 1 "4.7uF" V 8958 837 39  0000 L TNN
-F 2 "" H 9050 800 50  0001 C CNN
+F 2 "Capacitor_SMD:C_0805_2012Metric_Pad1.15x1.40mm_HandSolder" H 9050 800 50  0001 C CNN
 F 3 "~" H 9050 800 50  0001 C CNN
 	1    9050 800
@@
 F 0 "C19" V 12908 1212 39  0000 R TNN
 F 1 "4.7uF" V 12908 1287 39  0000 L TNN
-F 2 "" H 13000 1250 50  0001 C CNN
+F 2 "Capacitor_SMD:C_0805_2012Metric_Pad1.15x1.40mm_HandSolder" H 13000 1250 50  0001 C CNN
 F 3 "~" H 13000 1250 50  0001 C CNN
 	1    13000 1250
@@
 F 0 "C3" V 6258 2012 39  0000 R TNN
 F 1 "2.2uF" V 6258 2087 39  0000 L TNN
-F 2 "" H 6350 2050 50  0001 C CNN
+F 2 "Capacitor_SMD:C_0603_1608Metric_Pad1.05x0.95mm_HandSolder" H 6350 2050 50  0001 C CNN
 F 3 "~" H 6350 2050 50  0001 C CNN
 	1    6350 2050
@@
 F 0 "C1" V 6258 1912 39  0000 R TNN
 F 1 "2.2uF" V 6258 1987 39  0000 L TNN
-F 2 "" H 6350 1950 50  0001 C CNN
+F 2 "Capacitor_SMD:C_0603_1608Metric_Pad1.05x0.95mm_HandSolder" H 6350 1950 50  0001 C CNN
 F 3 "~" H 6350 1950 50  0001 C CNN
 	1    6350 1950
@@
 F 0 "C34" V 4158 5162 39  0000 R TNN
 F 1 "10pF" V 4158 5237 39  0000 L TNN
-F 2 "" H 4250 5200 50  0001 C CNN
+F 2 "Capacitor_SMD:C_0603_1608Metric_Pad1.05x0.95mm_HandSolder" H 4250 5200 50  0001 C CNN
 F 3 "~" H 4250 5200 50  0001 C CNN
 	1    4250 5200
@@
 F 0 "C33" V 3558 5162 39  0000 R TNN
 F 1 "10pF" V 3558 5237 39  0000 L TNN
-F 2 "" H 3650 5200 50  0001 C CNN
+F 2 "Capacitor_SMD:C_0603_1608Metric_Pad1.05x0.95mm_HandSolder" H 3650 5200 50  0001 C CNN
 F 3 "~" H 3650 5200 50  0001 C CNN
 	1    3650 5200
@@
 F 0 "JP1" H 12200 2835 50  0000 C CNN
 F 1 "Jumper_2_Open" H 12200 2744 50  0000 C CNN
-F 2 "" H 12200 2600 50  0001 C CNN
+F 2 "Connector_PinHeader_2.54mm:PinHeader_1x02_P2.54mm_Vertical" H 12200 2600 50  0001 C CNN
 F 3 "~" H 12200 2600 50  0001 C CNN
 	1    12200 2600
@@
 F 0 "JP2" H 12200 3085 50  0000 C CNN
 F 1 "Jumper_2_Open" H 12200 2994 50  0000 C CNN
-F 2 "" H 12200 2850 50  0001 C CNN
+F 2 "Connector_PinHeader_2.54mm:PinHeader_1x02_P2.54mm_Vertical" H 12200 2850 50  0001 C CNN
 F 3 "~" H 12200 2850 50  0001 C CNN
 	1    12200 2850
@@
 F 0 "J12" H 1807 3317 50  0000 C CNN
 F 1 "USB_B_Mini" H 1807 3226 50  0000 C CNN
-F 2 "" H 1900 2800 50  0001 C CNN
+F 2 "Connector_USB:USB_Mini-B_Wuerth_65100516121_Horizontal" H 1900 2800 50  0001 C CNN
 F 3 "~" H 1900 2800 50  0001 C CNN
 	1    1750 2850
@@
 F 0 "F5" V 2103 2650 50  0000 C CNN
 F 1 "500mA" V 2194 2650 50  0000 C CNN
-F 2 "" V 2230 2650 50  0001 C CNN
+F 2 "Fuse:Fuse_1206_3216Metric_Pad1.42x1.75mm_HandSolder" V 2230 2650 50  0001 C CNN
 F 3 "~" H 2300 2650 50  0001 C CNN
 	1    2300 2650
@@
 F 0 "J13" H 2400 6233 50  0000 C CNN
 F 1 "Micro_SD_Card" H 2400 6324 50  0000 C CNN
-F 2 "" H 3600 7350 50  0001 C CNN
+F 2 "Connector_Card:microSD_HC_Wuerth_693072010801" H 3600 7350 50  0001 C CNN
 F 3 "http://katalog.we-online.de/em/datasheet/693072010801.pdf" H 2450 7050 50  0001 C CNN
 	1    2450 7050
@@
 F 0 "EXP1" H 14250 3117 50  0000 C CNN
 F 1 "Conn_02x05_Odd_Even" H 14250 3026 50  0000 C CNN
-F 2 "" H 14200 2700 50  0001 C CNN
+F 2 "Connector_PinHeader_2.54mm:PinHeader_2x05_P2.54mm_Vertical" H 14200 2700 50  0001 C CNN
 F 3 "~" H 14200 2700 50  0001 C CNN
 	1    14200 2700
@@
 F 0 "EXP2" H 14250 4217 50  0000 C CNN
 F 1 "Conn_02x05_Odd_Even" H 14250 4126 50  0000 C CNN
-F 2 "" H 14200 3800 50  0001 C CNN
+F 2 "Connector_PinHeader_2.54mm:PinHeader_2x05_P2.54mm_Vertical" H 14200 3800 50  0001 C CNN
 F 3 "~" H 14200 3800 50  0001 C CNN
 	1    14200 3800
@@
 F 0 "UART1" H 12530 4392 50  0000 L CNN
 F 1 "Conn_01x04" H 12530 4301 50  0000 L CNN
-F 2 "" H 12450 4400 50  0001 C CNN
+F 2 "Connector_PinHeader_2.54mm:PinHeader_1x04_P2.54mm_Vertical" H 12450 4400 50  0001 C CNN
 F 3 "~" H 12450 4400 50  0001 C CNN
 	1    12450 4400
@@
 F 0 "SPI1" H 12400 5567 50  0000 C CNN
 F 1 "Conn_02x03_Odd_Even" H 12400 5476 50  0000 C CNN
-F 2 "" H 12350 5250 50  0001 C CNN
+F 2 "Connector_PinHeader_2.54mm:PinHeader_2x03_P2.54mm_Vertical" H 12350 5250 50  0001 C CNN
 F 3 "~" H 12350 5250 50  0001 C CNN
 	1    12350 5250
@@
 F 0 "I2C1" H 15130 4442 50  0000 L CNN
 F 1 "Conn_01x04" H 15130 4351 50  0000 L CNN
-F 2 "" H 15050 4450 50  0001 C CNN
+F 2 "Connector_PinHeader_2.54mm:PinHeader_1x04_P2.54mm_Vertical" H 15050 4450 50  0001 C CNN
 F 3 "~" H 15050 4450 50  0001 C CNN
 	1    15050 4450
@@
 F 0 "SWD1" H 13080 6992 50  0000 L CNN
 F 1 "Conn_01x05" H 13080 6901 50  0000 L CNN
-F 2 "" H 13000 6950 50  0001 C CNN
+F 2 "Connector_PinHeader_2.54mm:PinHeader_1x05_P2.54mm_Vertical" H 13000 6950 50  0001 C CNN
 F 3 "~" H 13000 6950 50  0001 C CNN
 	1    13000 6950
@@
 F 0 "J55" H 14700 8567 50  0000 C CNN
 F 1 "Conn_02x20_Odd_Even" H 14700 8476 50  0000 C CNN
-F 2 "" H 14650 7450 50  0001 C CNN
+F 2 "Connector_PinHeader_2.54mm:PinHeader_2x20_P2.54mm_Vertical" H 14650 7450 50  0001 C CNN
 F 3 "~" H 14650 7450 50  0001 C CNN
 	1    14650 7450
