File: Power.sch (KiCad schematic (older format))
At the start: 59 parts, among them J1 Conn_01x02, J2 Conn_01x02, U2 A4403, U3 TPS54531, U4 AP7361C-33E-13

Commit message: finished associating footprints with symbols
Parts:
- removed U2: A4403, Package_DFN_QFN:QFN-16-1EP_4x4mm_P0.65mm_EP2.7x2.7mm_ThermalVias, symbol Power~and~Buck~Converters:A4403
- removed U3: TPS54531, Package_SO:TI_SO-PowerPAD-8_ThermalVias, symbol Power~and~Buck~Converters:TPS54531
- removed U4: AP7361C-33E-13, Package_TO_SOT_SMD:SOT-223, symbol Power~and~Buck~Converters:AP7361C-33E-13
- added U2: A4403, Package_DFN_QFN:QFN-16-1EP_4x4mm_P0.65mm_EP2.7x2.7mm_ThermalVias, symbol Power_and_Buck_Converters:A4403
- added U3: TPS54531, Package_SO:TI_SO-PowerPAD-8_ThermalVias, symbol Power_and_Buck_Converters:TPS54531
- added U4: AP7361C-33E-13, Package_TO_SOT_SMD:SOT-223, symbol Power_and_Buck_Converters:AP7361C-33E-13
- J1, J2: footprint (none) -> TerminalBlock_Dinkle:TerminalBlock_Dinkle_DT-55-B01X-02_P10.00mm
Other:
- note added: "SOT-223\nNOT SOT-223R"
- note removed: "SOT-223\n"
Changed lines of the file:
@@
 F 0 "J1" H 1568 1125 50  0000 C CNN
 F 1 "Conn_01x02" H 1568 1216 50  0000 C CNN
-F 2 "" H 1650 1450 50  0001 C CNN
+F 2 "TerminalBlock_Dinkle:TerminalBlock_Dinkle_DT-55-B01X-02_P10.00mm" H 1650 1450 50  0001 C CNN
 F 3 "~" H 1650 1450 50  0001 C CNN
 	1    1650 1450
@@
 F 0 "J2" H 2568 1125 50  0000 C CNN
 F 1 "Conn_01x02" H 2568 1216 50  0000 C CNN
-F 2 "" H 2650 1450 50  0001 C CNN
+F 2 "TerminalBlock_Dinkle:TerminalBlock_Dinkle_DT-55-B01X-02_P10.00mm" H 2650 1450 50  0001 C CNN
 F 3 "~" H 2650 1450 50  0001 C CNN
 	1    2650 1450
@@
 	1350 2300 1550 2300
 Connection ~ 1550 2300
-$Comp
-L Power~and~Buck~Converters:A4403 U2
-U 1 1 5FB73845
-P 6750 1250
-F 0 "U2" H 6750 1665 50  0000 C CNN
-F 1 "A4403" H 6750 1574 50  0000 C CNN
-F 2 "Package_DFN_QFN:QFN-16-1EP_4x4mm_P0.65mm_EP2.7x2.7mm_ThermalVias" H 7200 450 50  0001 C CNN
-F 3 "" H 7200 450 50  0001 C CNN
-	1    6750 1250
-	1    0    0    -1
-$EndComp
-$Comp
-L Power~and~Buck~Converters:AP7361C-33E-13 U4
-U 1 1 5FB741EF
-P 6900 5950
-F 0 "U4" H 6900 6415 50  0000 C CNN
-F 1 "AP7361C-33E-13" H 6900 6324 50  0000 C CNN
-F 2 "Package_TO_SOT_SMD:SOT-223" H 7150 5850 50  0001 C CNN
-F 3 "" H 7150 5850 50  0001 C CNN
-	1    6900 5950
-	1    0    0    -1
-$EndComp
-$Comp
-L Power~and~Buck~Converters:TPS54531 U3
-U 1 1 5FB7478D
-P 6850 4000
-F 0 "U3" H 6850 4365 50  0000 C CNN
-F 1 "TPS54531" H 6850 4274 50  0000 C CNN
-F 2 "Package_SO:TI_SO-PowerPAD-8_ThermalVias" H 7200 3450 50  0001 C CNN
-F 3 "" H 7200 3450 50  0001 C CNN
-	1    6850 4000
-	1    0    0    -1
-$EndComp
 Text GLabel 4550 3900 0    50   Input ~ 0
 VIN_FUSED
@@
 IHLP2525EZER4R7M01
 Text Notes 7050 5400 0    50   ~ 0
-SOT-223\n
+SOT-223\nNOT SOT-223R
+$Comp
+L Power_and_Buck_Converters:A4403 U2
+U 1 1 5FB2EF5D
+P 6750 1250
+F 0 "U2" H 6750 1665 50  0000 C CNN
+F 1 "A4403" H 6750 1574 50  0000 C CNN
+F 2 "Package_DFN_QFN:QFN-16-1EP_4x4mm_P0.65mm_EP2.7x2.7mm_ThermalVias" H 7200 450 50  0001 C CNN
+F 3 "" H 7200 450 50  0001 C CNN
+	1    6750 1250
+	1    0    0    -1
+$EndComp
+$Comp
+L Power_and_Buck_Converters:AP7361C-33E-13 U4
+U 1 1 5FB2FC89
+P 6900 5950
+F 0 "U4" H 6900 6415 50  0000 C CNN
+F 1 "AP7361C-33E-13" H 6900 6324 50  0000 C CNN
+F 2 "Package_TO_SOT_SMD:SOT-223" H 7150 5850 50  0001 C CNN
+F 3 "" H 7150 5850 50  0001 C CNN
+	1    6900 5950
+	1    0    0    -1
+$EndComp
+$Comp
+L Power_and_Buck_Converters:TPS54531 U3
+U 1 1 5FB30DE4
+P 6850 4000
+F 0 "U3" H 6850 4365 50  0000 C CNN
+F 1 "TPS54531" H 6850 4274 50  0000 C CNN
+F 2 "Package_SO:TI_SO-PowerPAD-8_ThermalVias" H 7200 3450 50  0001 C CNN
+F 3 "" H 7200 3450 50  0001 C CNN
+	1    6850 4000
+	1    0    0    -1
+$EndComp
 $EndSCHEMATC
