File: Stepper Drivers 2.sch (KiCad schematic (older format))
At the start: 88 parts, among them J10 Conn_01x04, J7 Conn_01x04, J8 Conn_01x04, J9 Conn_01x04

Commit message: Added more footprints
Parts:
- E1_Driver1, E2_Driver1, E3_Driver1, E4_Driver1: footprint (none) -> Package_DFN_QFN:QFN-28-1EP_5x5mm_P0.5mm_EP3.35x3.35mm_ThermalVias
- R46, R47, R54, R55: footprint (none) -> Resistor_SMD:R_0603_1608Metric_Pad1.05x0.95mm_HandSolder
- R48, R49, R50, R51, R52, R53, R56, R57, R58, R59, R60, R61: footprint (none) -> Resistor_SMD:R_0805_2012Metric_Pad1.15x1.40mm_HandSolder
Changed lines of the file:
@@
 F 0 "E1_Driver1" H 2650 2665 50  0000 C CNN
 F 1 "TMC2209" H 2650 2574 50  0000 C CNN
-F 2 "" H 2750 1850 50  0001 C CNN
+F 2 "Package_DFN_QFN:QFN-28-1EP_5x5mm_P0.5mm_EP3.35x3.35mm_ThermalVias" H 2750 1850 50  0001 C CNN
 F 3 "" H 2750 1850 50  0001 C CNN
 	1    2650 1850
@@
 F 0 "R51" V 3968 2646 39  0000 L BNN
 F 1 "0R11" V 3968 2555 39  0000 R BNN
-F 2 "" H 3900 2600 50  0001 C CNN
+F 2 "Resistor_SMD:R_0805_2012Metric_Pad1.15x1.40mm_HandSolder" H 3900 2600 50  0001 C CNN
 F 3 "~" H 3900 2600 50  0001 C CNN
 	1    3900 2600
@@
 F 0 "R53" V 4268 2646 39  0000 L BNN
 F 1 "0R11" V 4268 2555 39  0000 R BNN
-F 2 "" H 4200 2600 50  0001 C CNN
+F 2 "Resistor_SMD:R_0805_2012Metric_Pad1.15x1.40mm_HandSolder" H 4200 2600 50  0001 C CNN
 F 3 "~" H 4200 2600 50  0001 C CNN
 	1    4200 2600
@@
 F 0 "R49" V 1418 2446 39  0000 L BNN
 F 1 "0R11" V 1418 2355 39  0000 R BNN
-F 2 "" H 1350 2400 50  0001 C CNN
+F 2 "Resistor_SMD:R_0805_2012Metric_Pad1.15x1.40mm_HandSolder" H 1350 2400 50  0001 C CNN
 F 3 "~" H 1350 2400 50  0001 C CNN
 	1    1350 2400
@@
 F 0 "R47" V 1218 1496 39  0000 L BNN
 F 1 "20k" V 1218 1405 39  0000 R BNN
-F 2 "" H 1150 1450 50  0001 C CNN
+F 2 "Resistor_SMD:R_0603_1608Metric_Pad1.05x0.95mm_HandSolder" H 1150 1450 50  0001 C CNN
 F 3 "~" H 1150 1450 50  0001 C CNN
 	1    1150 1450
@@
 F 0 "E2_Driver1" H 8000 2665 50  0000 C CNN
 F 1 "TMC2209" H 8000 2574 50  0000 C CNN
-F 2 "" H 8100 1850 50  0001 C CNN
+F 2 "Package_DFN_QFN:QFN-28-1EP_5x5mm_P0.5mm_EP3.35x3.35mm_ThermalVias" H 8100 1850 50  0001 C CNN
 F 3 "" H 8100 1850 50  0001 C CNN
 	1    8000 1850
@@
 F 0 "R58" V 9318 2646 39  0000 L BNN
 F 1 "0R11" V 9318 2555 39  0000 R BNN
-F 2 "" H 9250 2600 50  0001 C CNN
+F 2 "Resistor_SMD:R_0805_2012Metric_Pad1.15x1.40mm_HandSolder" H 9250 2600 50  0001 C CNN
 F 3 "~" H 9250 2600 50  0001 C CNN
 	1    9250 2600
@@
 F 0 "R60" V 9618 2646 39  0000 L BNN
 F 1 "0R11" V 9618 2555 39  0000 R BNN
-F 2 "" H 9550 2600 50  0001 C CNN
+F 2 "Resistor_SMD:R_0805_2012Metric_Pad1.15x1.40mm_HandSolder" H 9550 2600 50  0001 C CNN
 F 3 "~" H 9550 2600 50  0001 C CNN
 	1    9550 2600
@@
 F 0 "R56" V 6768 2446 39  0000 L BNN
 F 1 "0R11" V 6768 2355 39  0000 R BNN
-F 2 "" H 6700 2400 50  0001 C CNN
+F 2 "Resistor_SMD:R_0805_2012Metric_Pad1.15x1.40mm_HandSolder" H 6700 2400 50  0001 C CNN
 F 3 "~" H 6700 2400 50  0001 C CNN
 	1    6700 2400
@@
 F 0 "R54" V 6568 1496 39  0000 L BNN
 F 1 "20k" V 6568 1405 39  0000 R BNN
-F 2 "" H 6500 1450 50  0001 C CNN
+F 2 "Resistor_SMD:R_0603_1608Metric_Pad1.05x0.95mm_HandSolder" H 6500 1450 50  0001 C CNN
 F 3 "~" H 6500 1450 50  0001 C CNN
 	1    6500 1450
@@
 F 0 "E3_Driver1" H 2600 5615 50  0000 C CNN
 F 1 "TMC2209" H 2600 5524 50  0000 C CNN
-F 2 "" H 2700 4800 50  0001 C CNN
+F 2 "Package_DFN_QFN:QFN-28-1EP_5x5mm_P0.5mm_EP3.35x3.35mm_ThermalVias" H 2700 4800 50  0001 C CNN
 F 3 "" H 2700 4800 50  0001 C CNN
 	1    2600 4800
@@
 F 0 "R50" V 3918 5596 39  0000 L BNN
 F 1 "0R11" V 3918 5505 39  0000 R BNN
-F 2 "" H 3850 5550 50  0001 C CNN
+F 2 "Resistor_SMD:R_0805_2012Metric_Pad1.15x1.40mm_HandSolder" H 3850 5550 50  0001 C CNN
 F 3 "~" H 3850 5550 50  0001 C CNN
 	1    3850 5550
@@
 F 0 "R52" V 4218 5596 39  0000 L BNN
 F 1 "0R11" V 4218 5505 39  0000 R BNN
-F 2 "" H 4150 5550 50  0001 C CNN
+F 2 "Resistor_SMD:R_0805_2012Metric_Pad1.15x1.40mm_HandSolder" H 4150 5550 50  0001 C CNN
 F 3 "~" H 4150 5550 50  0001 C CNN
 	1    4150 5550
@@
 F 0 "R48" V 1368 5396 39  0000 L BNN
 F 1 "0R11" V 1368 5305 39  0000 R BNN
-F 2 "" H 1300 5350 50  0001 C CNN
+F 2 "Resistor_SMD:R_0805_2012Metric_Pad1.15x1.40mm_HandSolder" H 1300 5350 50  0001 C CNN
 F 3 "~" H 1300 5350 50  0001 C CNN
 	1    1300 5350
@@
 F 0 "R46" V 1168 4446 39  0000 L BNN
 F 1 "20k" V 1168 4355 39  0000 R BNN
-F 2 "" H 1100 4400 50  0001 C CNN
+F 2 "Resistor_SMD:R_0603_1608Metric_Pad1.05x0.95mm_HandSolder" H 1100 4400 50  0001 C CNN
 F 3 "~" H 1100 4400 50  0001 C CNN
 	1    1100 4400
@@
 F 0 "R59" V 9318 5596 39  0000 L BNN
 F 1 "0R11" V 9318 5505 39  0000 R BNN
-F 2 "" H 9250 5550 50  0001 C CNN
+F 2 "Resistor_SMD:R_0805_2012Metric_Pad1.15x1.40mm_HandSolder" H 9250 5550 50  0001 C CNN
 F 3 "~" H 9250 5550 50  0001 C CNN
 	1    9250 5550
@@
 F 0 "R61" V 9618 5596 39  0000 L BNN
 F 1 "0R11" V 9618 5505 39  0000 R BNN
-F 2 "" H 9550 5550 50  0001 C CNN
+F 2 "Resistor_SMD:R_0805_2012Metric_Pad1.15x1.40mm_HandSolder" H 9550 5550 50  0001 C CNN
 F 3 "~" H 9550 5550 50  0001 C CNN
 	1    9550 5550
@@
 F 0 "R57" V 6768 5396 39  0000 L BNN
 F 1 "0R11" V 6768 5305 39  0000 R BNN
-F 2 "" H 6700 5350 50  0001 C CNN
+F 2 "Resistor_SMD:R_0805_2012Metric_Pad1.15x1.40mm_HandSolder" H 6700 5350 50  0001 C CNN
 F 3 "~" H 6700 5350 50  0001 C CNN
 	1    6700 5350
@@
 F 0 "R55" V 6568 4446 39  0000 L BNN
 F 1 "20k" V 6568 4355 39  0000 R BNN
-F 2 "" H 6500 4400 50  0001 C CNN
+F 2 "Resistor_SMD:R_0603_1608Metric_Pad1.05x0.95mm_HandSolder" H 6500 4400 50  0001 C CNN
 F 3 "~" H 6500 4400 50  0001 C CNN
 	1    6500 4400
@@
 F 0 "E4_Driver1" H 8000 5615 50  0000 C CNN
 F 1 "TMC2209" H 8000 5524 50  0000 C CNN
-F 2 "" H 8100 4800 50  0001 C CNN
+F 2 "Package_DFN_QFN:QFN-28-1EP_5x5mm_P0.5mm_EP3.35x3.35mm_ThermalVias" H 8100 4800 50  0001 C CNN
 F 3 "" H 8100 4800 50  0001 C CNN
 	1    8000 4800

Commit message: started some routing
Parts:
- JP14, JP15, JP18, JP19: footprint Connector_PinHeader_2.54mm:PinHeader_1x03_P2.54mm_Vertical -> Jumper:SolderJumper-3_P1.3mm_Open_RoundedPad1.0x1.5mm
Changed lines of the file:
@@
 F 0 "JP15" H 3350 3163 50  0000 C CNN
 F 1 "SPREAD_STEALTH" H 3200 3250 50  0000 C CNN
-F 2 "Connector_PinHeader_2.54mm:PinHeader_1x03_P2.54mm_Vertical" H 3350 3050 50  0001 C CNN
+F 2 "Jumper:SolderJumper-3_P1.3mm_Open_RoundedPad1.0x1.5mm" H 3350 3050 50  0001 C CNN
 F 3 "~" H 3350 3050 50  0001 C CNN
 	1    3350 3050
@@
 F 0 "JP14" H 3300 6113 50  0000 C CNN
 F 1 "SPREAD_STEALTH" H 3150 6200 50  0000 C CNN
-F 2 "Connector_PinHeader_2.54mm:PinHeader_1x03_P2.54mm_Vertical" H 3300 6000 50  0001 C CNN
+F 2 "Jumper:SolderJumper-3_P1.3mm_Open_RoundedPad1.0x1.5mm" H 3300 6000 50  0001 C CNN
 F 3 "~" H 3300 6000 50  0001 C CNN
 	1    3300 6000
@@
 F 0 "JP18" H 8700 3163 50  0000 C CNN
 F 1 "SPREAD_STEALTH" H 8550 3250 50  0000 C CNN
-F 2 "Connector_PinHeader_2.54mm:PinHeader_1x03_P2.54mm_Vertical" H 8700 3050 50  0001 C CNN
+F 2 "Jumper:SolderJumper-3_P1.3mm_Open_RoundedPad1.0x1.5mm" H 8700 3050 50  0001 C CNN
 F 3 "~" H 8700 3050 50  0001 C CNN
 	1    8700 3050
@@
 F 0 "JP19" H 8700 6113 50  0000 C CNN
 F 1 "SPREAD_STEALTH" H 8550 6200 50  0000 C CNN
-F 2 "Connector_PinHeader_2.54mm:PinHeader_1x03_P2.54mm_Vertical" H 8700 6000 50  0001 C CNN
+F 2 "Jumper:SolderJumper-3_P1.3mm_Open_RoundedPad1.0x1.5mm" H 8700 6000 50  0001 C CNN
 F 3 "~" H 8700 6000 50  0001 C CNN
 	1    8700 6000
