File: Board.kicad_pcb (KiCad board)
At the start: 2 copper layers, 511 parts, among them J1 MAIN_POWER, J10 Conn_01x04, J11 Conn_01x04, J12 USB_B_Mini, J13 Micro_SD_Card, J14 Conn_02x03_Odd_Even, J15 Conn_02x03_Odd_Even, J16 H0, J17 H4, J18 F0, J19 F4, J2 BED_POWER, J20 Conn_02x03_Odd_Even, J21 Conn_02x03_Odd_Even, J22 H1, J23 H5, J24 F1, J25 F5, J26 Conn_02x03_Odd_Even, J27 Conn_02x03_Odd_Even, J28 H2, J29 HC, J3 Conn_01x04, J30 F2, J31 F6, J32 Conn_02x03_Odd_Even, J33 Conn_02x03_Odd_Even, J34 H3, J35 HB, J36 F3, J37 F7, J38 Conn_01x03, J39 Conn_01x03, J4 Conn_01x04, J40 Conn_01x03, J41 Conn_01x03, J42 Conn_01x03, J43 Conn_01x03, J44 Conn_01x03, J45 Conn_01x03, J46 Conn_01x03, J47 Conn_01x02, J48 Conn_01x02, J49 Conn_01x02, J5 Conn_01x04, J50 Conn_01x02, J51 Conn_01x02, J52 Conn_01x02, J53 Conn_01x02, J54 Conn_01x02, J55 Conn_02x20_Odd_Even, J6 Conn_01x04, J7 Conn_01x04, J8 Conn_01x04, J9 Conn_01x04, Q1 Q_NMOS_GDS, Q10 Q_NMOS_GDS, Q11 Q_NMOS_GSD, Q12 Q_NMOS_GSD, Q13 Q_NMOS_GDS, Q14 Q_NMOS_GDS, Q15 Q_NMOS_GSD, Q16 Q_NMOS_GSD, Q2 Q_NMOS_GDS, Q3 Q_NMOS_GSD, Q4 Q_NMOS_GSD, Q5 Q_NMOS_GDS, Q6 Q_NMOS_GDS, Q7 Q_NMOS_GSD, Q8 Q_NMOS_GSD, Q9 Q_NMOS_GDS, SW1 SW_Push, U1 STM32F407IGTx, U2 A4403, U3 TPS54531, U4 AP7361C-33E-13, U5 74HCT245, U6 74HCT245, U7 24C02, Y1 12MHz, 20pF

Commit message: Roughtly Layed out power converters and FETs
Parts:
- moved C47 342.6 mm to (53.9, 112.3), turned to 180 degrees
- moved C39 336.5 mm to (55.4, 108.8)
- moved D9 326.9 mm to (143.4, 130.8), turned to 90 degrees
- moved D15 326.5 mm to (131.9, 130.9), turned to 90 degrees
- moved D16 326.3 mm to (86.2, 130.9), turned to 90 degrees
- moved R85 325.0 mm to (143.4, 134.3), turned to 270 degrees
- moved R97 319.8 mm to (120.6, 134.3), turned to 270 degrees
- moved R86 318.9 mm to (97.7, 134.2), turned to 270 degrees
- moved R87 316.2 mm to (138.6, 123.1), turned to 90 degrees
- moved R88 315.3 mm to (92.8, 123.1), turned to 90 degrees
- moved R8 313.0 mm to (79.6, 86.0)
- moved R92 310.8 mm to (86.2, 134.3), turned to 270 degrees
- moved R93 304.3 mm to (127.2, 123.0), turned to 90 degrees
- moved R94 301.0 mm to (56.6, 122.6), turned to 90 degrees
- moved R100 295.3 mm to (76.4, 122.6), turned to 90 degrees
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Connections:
- R8 pad 1: Net-(C45-Pad1) -> Net-(D4-Pad2)
- R9 pad 1: Net-(C45-Pad1) -> Net-(D4-Pad2)

Commit message: started some routing
Parts:
- JP10, JP11, JP14, JP15, JP18, JP19, JP21, JP6, JP7: footprint Connector_PinHeader_2.54mm:PinHeader_1x03_P2.54mm_Vertical -> Jumper:SolderJumper-3_P1.3mm_Open_RoundedPad1.0x1.5mm
- moved H2 287.1 mm to (160.6, 146.8)
- moved C177 45.4 mm to (-21.0, -40.9), turned to 180 degrees
- moved R65 41.7 mm to (-20.8, -39.1), turned to 180 degrees
- moved C172 36.8 mm to (-24.1, -54.0), turned to 90 degrees
- moved C178 36.4 mm to (-16.5, -60.7), turned to 270 degrees
- moved C168 34.6 mm to (-19.4, -50.4), turned to 90 degrees
- moved C174 32.2 mm to (-10.5, -41.2), turned to 270 degrees
- moved C179 28.9 mm to (-19.2, -61.6), turned to 180 degrees
- moved R63 25.3 mm to (-17.1, -52.3), turned to 90 degrees
- moved C181 24.7 mm to (-11.3, -61.6)
- moved R64 23.9 mm to (-12.2, -41.0), turned to 270 degrees
- moved C175 22.7 mm to (-20.7, -43.7), turned to 180 degrees
- moved C176 20.8 mm to (-9.00, -41.2), turned to 270 degrees
- moved C171 20.1 mm to (-9.78, -47.9), turned to 180 degrees
- moved C169 19.2 mm to (-13.0, -53.3)
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Routing:
- net GND: track 0.00 -> 247.2 mm
- net VIN_FUSED: track 0.00 -> 212.3 mm
- net VIN_BED_FUSED: track 0.00 -> 114.8 mm
- net VIN: track 0.00 -> 54.7 mm
- net Net-(C44-Pad1): track 0.00 -> 33.6 mm
- net Net-(C47-Pad1): track 0.00 -> 30.2 mm
- net Net-(D4-Pad2): track 0.00 -> 24.9 mm, vias 0 -> 2
- net Net-(D26-Pad1): track 0.00 -> 22.8 mm
- net Net-(D32-Pad1): track 0.00 -> 22.6 mm
- net Net-(D20-Pad1): track 0.00 -> 22.6 mm
- net Net-(D14-Pad1): track 0.00 -> 22.6 mm
- net Net-(D25-Pad1): track 0.00 -> 22.6 mm
- net Net-(D19-Pad1): track 0.00 -> 22.6 mm
- net Net-(D13-Pad1): track 0.00 -> 22.6 mm
- net Net-(D31-Pad1): track 0.00 -> 22.6 mm
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Other:
- copper layers 2 -> 4

Commit message: small component placement
Parts:
- moved JP9 382.4 mm to (-152.2, 60.6)
- moved C98 352.4 mm to (-159.3, -30.9)
- moved E0_Driver1 343.6 mm to (-132.8, 51.1), turned to 180 degrees
- moved C92 343.2 mm to (-168.0, -30.3)
- moved JP5 336.7 mm to (-103.5, 69.5)
- moved X_Driver1 328.5 mm to (-101.3, 50.5), turned to 180 degrees
- moved JP11 328.3 mm to (-123.3, 44.0)
- moved J6 312.6 mm to (-133.8, 34.8)
- moved C90 311.1 mm to (-166.6, -22.3)
- moved J4 300.6 mm to (-104.9, 38.0)
- moved JP7 297.6 mm to (-90.5, 45.0)
- moved JP10 285.4 mm to (-55.9, 45.8)
- moved JP8 279.7 mm to (-64.9, 66.2)
- moved Y_Driver1 265.2 mm to (-64.7, 51.0), turned to 180 degrees
- moved JP4 259.6 mm to (-24.9, 64.8)
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
Commit message: routed mosfets and buffers
Parts:
- moved C90 150.7 mm to (-16.0, -26.3)
- moved C92 150.7 mm to (-17.4, -34.4)
- moved C98 150.7 mm to (-8.68, -35.0)
- moved J4 133.0 mm to (-56.4, -85.9)
- moved J5 133.0 mm to (-20.9, -88.1)
- moved JP10 133.0 mm to (-7.38, -78.0)
- moved JP5 133.0 mm to (-55.0, -54.4)
- moved JP7 133.0 mm to (-42.0, -78.9)
- moved JP8 133.0 mm to (-16.4, -57.7)
- moved X_Driver1 133.0 mm to (-52.9, -73.4)
- moved Y_Driver1 133.0 mm to (-16.2, -72.9)
- moved J6 120.5 mm to (-98.7, -80.5)
- moved E0_Driver1 119.9 mm to (-95.3, -62.8)
- moved JP11 119.9 mm to (-85.9, -69.9)
- moved JP9 119.9 mm to (-114.8, -53.2)
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Routing:
- net GND: track 247.2 -> 351.7 mm
- net FAN0_BUFF: track 0.00 -> 86.9 mm
- net FAN1_BUFF: track 0.00 -> 81.1 mm
- net FAN2_BUFF: track 0.00 -> 76.0 mm
- net FAN7_BUFF: track 0.00 -> 70.2 mm
- net FAN3_BUFF: track 0.00 -> 70.1 mm
- net FAN4_BUFF: track 0.00 -> 64.3 mm
- net FAN6_BUFF: track 0.00 -> 60.9 mm
- net FAN5_BUFF: track 0.00 -> 58.4 mm
- net HEATER0_BUFF: track 0.00 -> 55.4 mm
- net CHAMBER_HEATER_BUFF: track 0.00 -> 45.9 mm
- net HEATER1_BUFF: track 0.00 -> 45.2 mm
- net HEATER2_BUFF: track 0.00 -> 35.4 mm
- net BED_HEATER_BUFF: track 0.00 -> 31.6 mm
- net +5V: track 7.84 -> 33.6 mm
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